File: Models/TransimpedanceAmplifier/DUT.kicad_sch (KiCad schematic)
At the start: 0 parts

Commit message: Labeled all the input/output nodes of the power subsystems
Other:
- note added: "TODO: List all devices that will be tested Gather their symbols and purchase links Exclude them from the PCB"
Changed lines of the file:
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@@
 	(generator_version "9.0")
 	(paper "A4")
+	(text "TODO: List all devices that will be tested\nGather their symbols and purchase links\nExclude them from the PCB"
+		(exclude_from_sim no)
+		(at 102.108 52.07 0)
+		(effects
+			(font
+				(size 1.27 1.27)
+			)
+			(justify left top)
+		)
+	)
 )

Commit message: Next step is to refactor the power net at each op-amp
Other:
- note removed: "TODO: List all devices that will be tested Gather their symbols and purchase links Exclude them from the PCB"
Changed lines of the file:
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@@
 	(generator_version "9.0")
 	(paper "A4")
-	(text "TODO: List all devices that will be tested\nGather their symbols and purchase links\nExclude them from the PCB"
-		(exclude_from_sim no)
-		(at 102.108 52.07 0)
-		(effects
-			(font
-				(size 1.27 1.27)
-			)
-			(justify left top)
-		)
-	)
 )
