File: Models/TransimpedanceAmplifier/Teensy.kicad_sch (KiCad schematic)
At the start: 5 parts, among them J11 Conn_01x24_Pin, J13 Conn_01x24_Pin, U13 Teensy4.1

Commit message: Save progress
Other:
- note added: "All 3.3V pins are electrically equivalent. They connect to the same net in the Teensy 4.1 PCB schematic. In theory, I can draw 250 mA out of any one of them. Their physical separation is mostly an issue at high frequencies, where local decoupling networks are used anyway. The same should be true about GND pins. To simplify everything, I'll connect all GND pins to my PCB and tie them into the same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"
- note added: "Connected to low-cost Windows PC through Micro-USB port: 49 (VUSB) 66 (D-) 67 (D+) GND"
- note removed: "Connected to low-cost Windows PC: 49 (VUSB) 66 (D-) 67 (D+) GND"
- moved on the sheet: J11, J13, J_Teensy_Left, J_Teensy_Right, U13
Changed lines of the file:
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@@
 	(generator_version "9.0")
 	(paper "A4")
-	(text "Connected to low-cost Windows PC:\n\n49 (VUSB)\n66 (D-)\n67 (D+)\nGND"
+	(text "Connected to low-cost Windows PC\nthrough Micro-USB port:\n\n49 (VUSB)\n66 (D-)\n67 (D+)\nGND"
 		(exclude_from_sim no)
-		(at 134.62 32.258 0)
+		(at 127.254 45.466 0)
 		(effects
 			(font
@@
 		)
 	)
-	(no_connect
-		(at 127 129.54)
-	)
-	(no_connect
-		(at 158.75 144.78)
-	)
-	(no_connect
-		(at 127 120.65)
-	)
-	(no_connect
-		(at 147.32 144.78)
-	)
-	(no_connect
-		(at 208.28 57.15)
-	)
-	(no_connect
-		(at 182.88 132.08)
-	)
-	(no_connect
-		(at 182.88 53.34)
-	)
-	(no_connect
-		(at 182.88 121.92)
-	)
-	(no_connect
-		(at 182.88 134.62)
-	)
-	(no_connect
-		(at 127 127)
-	)
-	(no_connect
-		(at 151.13 144.78)
-	)
-	(no_connect
-		(at 127 134.62)
-	)
-	(no_connect
-		(at 127 137.16)
-	)
-	(no_connect
-		(at 162.56 144.78)
-	)
-	(no_connect
-		(at 182.88 127)
-	)
-	(no_connect
-		(at 182.88 124.46)
-	)
-	(no_connect
-		(at 182.88 129.54)
-	)
-	(no_connect
-		(at 127 132.08)
-	)
-	(no_connect
-		(at 154.94 144.78)
-	)
-	(no_connect
-		(at 127 123.19)
-	)
-	(hierarchical_label "CS_DAC"
-		(shape output)
-		(at 208.28 107.95 0)
+	(text "All 3.3V pins are electrically equivalent. They connect to the same\nnet in the Teensy 4.1 PCB schematic. In theory, I can draw 250 mA out\nof any one of them. Their physical separation is mostly an issue at\nhigh frequencies, where local decoupling networks are used anyway.\n\nThe same should be true about GND pins. To simplify everything, I'll\nconnect all GND pins to my PCB and tie them into the same net."
+		(exclude_from_sim no)
+		(at 190.754 39.116 0)
 		(effects
 			(font
 				(size 1.27 1.27)
 			)
-			(justify left)
-		)
-	)
-	(hierarchical_label "CS_ADC"
+			(justify left top)
+		)
+	)
+	(no_connect
+		(at 76.2 142.24)
+	)
+	(no_connect
+		(at 107.95 157.48)
+	)
+	(no_connect
+		(at 76.2 133.35)
+	)
+	(no_connect
+		(at 96.52 157.48)
+	)
+	(no_connect
+		(at 157.48 69.85)
+	)
+	(no_connect
+		(at 132.08 144.78)
+	)
+	(no_connect
+		(at 132.08 66.04)
+	)
+	(no_connect
+		(at 132.08 134.62)
+	)
+	(no_connect
+		(at 132.08 147.32)
+	)
+	(no_connect
+		(at 76.2 139.7)
+	)
+	(no_connect
+		(at 100.33 157.48)
+	)
+	(no_connect
+		(at 76.2 147.32)
+	)
+	(no_connect
+		(at 76.2 149.86)
+	)
+	(no_connect
+		(at 111.76 157.48)
+	)
+	(no_connect
+		(at 132.08 139.7)
+	)
+	(no_connect
+		(at 132.08 137.16)
+	)
+	(no_connect
+		(at 132.08 142.24)
+	)
+	(no_connect
+		(at 76.2 144.78)
+	)
+	(no_connect
+		(at 104.14 157.48)
+	)
+	(no_connect
+		(at 76.2 135.89)
+	)
+	(hierarchical_label "CS_DAC"
 		(shape output)
-		(at 208.28 105.41 0)
+		(at 157.48 120.65 0)
 		(effects
 			(font
@@
 		)
 	)
-	(hierarchical_label "SCK"
+	(hierarchical_label "CS_ADC"
 		(shape output)
-		(at 208.28 90.17 0)
+		(at 157.48 118.11 0)
 		(effects
 			(font
@@
 		)
 	)
-	(hierarchical_label "MOSI"
+	(hierarchical_label "SCK"
 		(shape output)
-		(at 101.6 87.63 180)
+		(at 157.48 102.87 0)
 		(effects
 			(font
 				(size 1.27 1.27)
 			)
-			(justify right)
-		)
-	)
-	(hierarchical_label "MISO"
-		(shape input)
-		(at 101.6 90.17 180)
+			(justify left)
+		)
+	)
+	(hierarchical_label "MOSI"
+		(shape output)
+		(at 50.8 100.33 180)
 		(effects
 			(font
@@
 		)
 	)
+	(hierarchical_label "MISO"
+		(shape input)
+		(at 50.8 102.87 180)
+		(effects
+			(font
+				(size 1.27 1.27)
+			)
+			(justify right)
+		)
+	)
 	(symbol
 		(lib_id "Connector:Conn_01x24_Socket")
-		(at 203.2 87.63 180)
+		(at 152.4 100.33 180)
 		(unit 1)
 		(exclude_from_sim no)
@@
 		(dnp no)
 		(property "Reference" "J_Teensy_Right"
-			(at 209.55 48.768 0)
+			(at 158.75 61.468 0)
 			(effects
 				(font
@@
 		)
 		(property "Value" "Conn_01x24_Socket"
-			(at 212.09 51.562 0)
+			(at 161.29 64.262 0)
 			(effects
 				(font
@@
 		)
 		(property "Footprint" ""
-			(at 203.2 87.63 0)
+			(at 152.4 100.33 0)
 			(effects
 				(font
@@
 		)
 		(property "Datasheet" "~"
-			(at 203.2 87.63 0)
+			(at 152.4 100.33 0)
 			(effects
 				(font
@@
 		)
 		(property "Description" "Generic connector, single row, 01x24, script generated"
-			(at 203.2 87.63 0)
+			(at 152.4 100.33 0)
 			(effects
 				(font
@@
 		)
 		(property "Purchase Link" "https://www.digikey.com/en/products/detail/sullins-connector-solutions/PPPC241LFBN-RC/810196"
-			(at 203.2 87.63 0)
+			(at 152.4 100.33 0)
 			(effects
 				(font
@@
 	(symbol
 		(lib_id "Connector:Conn_01x24_Socket")
-		(at 106.68 85.09 0)
+		(at 55.88 97.79 0)
 		(unit 1)
 		(exclude_from_sim no)
@@
 		(dnp no)
 		(property "Reference" "J_Teensy_Left"
-			(at 93.98 50.546 0)
+			(at 43.18 63.246 0)
 			(effects
 				(font
@@
 		)
 		(property "Value" "Conn_01x24_Socket"
-			(at 87.884 53.086 0)
+			(at 37.084 65.786 0)
 			(effects
 				(font
@@
 		)
 		(property "Footprint" ""
-			(at 106.68 85.09 0)
+			(at 55.88 97.79 0)
 			(effects
 				(font
@@
 		)
 		(property "Datasheet" "~"
-			(at 106.68 85.09 0)
+			(at 55.88 97.79 0)
 			(effects
 				(font
@@
 		)
 		(property "Description" "Generic connector, single row, 01x24, script generated"
-			(at 106.68 85.09 0)
+			(at 55.88 97.79 0)
 			(effects
 				(font
@@
 		)
 		(property "Purchase Link" "https://www.digikey.com/en/products/detail/sullins-connector-solutions/PPPC241LFBN-RC/810196"
-			(at 106.68 85.09 0)
+			(at 55.88 97.79 0)
 			(effects
 				(font
@@
 	(symbol
 		(lib_id "Connector:Conn_01x24_Pin")
-		(at 121.92 85.09 0)
+		(at 71.12 97.79 0)
 		(unit 1)
 		(exclude_from_sim no)
 		(in_bom yes)
-		(on_board yes)
+		(on_board no)
 		(dnp no)
 		(property "Reference" "J13"
-			(at 125.222 50.038 0)
+			(at 74.422 62.738 0)
 			(effects
 				(font
@@
 		)
 		(property "Value" "Conn_01x24_Pin"
-			(at 119.126 53.086 0)
+			(at 68.326 65.786 0)
 			(effects
 				(font
@@
 		)
 		(property "Footprint" ""
-			(at 121.92 85.09 0)
+			(at 71.12 97.79 0)
 			(effects
 				(font
@@
 		)
 		(property "Datasheet" "~"
-			(at 121.92 85.09 0)
+			(at 71.12 97.79 0)
 			(effects
 				(font
@@
 		)
 		(property "Description" "Generic connector, single row, 01x24, script generated"
-			(at 121.92 85.09 0)
+			(at 71.12 97.79 0)
 			(effects
 				(font
@@
 		)
 		(property "Purchase Link" "https://www.digikey.com/en/products/detail/sullins-connector-solutions/PRPC024SAAN-RC/2775230"
-			(at 121.92 85.09 0)
+			(at 71.12 97.79 0)
 			(effects
 				(font
@@
 	(symbol
 		(lib_id "Connector:Conn_01x24_Pin")
-		(at 187.96 87.63 180)
+		(at 137.16 100.33 180)
 		(unit 1)
 		(exclude_from_sim no)
 		(in_bom yes)
-		(on_board yes)
+		(on_board no)
 		(dnp no)
 		(property "Reference" "J11"
-			(at 185.166 50.292 0)
+			(at 134.366 62.992 0)
 			(effects
 				(font
@@
 		)
 		(property "Value" "Conn_01x24_Pin"
-			(at 185.166 52.832 0)
+			(at 134.366 65.532 0)
 			(effects
 				(font
@@
 		)
 		(property "Footprint" ""
-			(at 187.96 87.63 0)
+			(at 137.16 100.33 0)
 			(effects
 				(font
@@
 		)
 		(property "Datasheet" "~"
-			(at 187.96 87.63 0)
+			(at 137.16 100.33 0)
 			(effects
 				(font
@@
 		)
 		(property "Description" "Generic connector, single row, 01x24, script generated"
-			(at 187.96 87.63 0)
+			(at 137.16 100.33 0)
 			(effects
 				(font
@@
 		)
 		(property "Purchase Link" "https://www.digikey.com/en/products/detail/sullins-connector-solutions/PRPC024SAAN-RC/2775230"
-			(at 187.96 87.63 0)
+			(at 137.16 100.33 0)
 			(effects
 				(font
@@
 	(symbol
 		(lib_id "teensy:Teensy4.1")
-		(at 154.94 111.76 0)
+		(at 104.14 124.46 0)
 		(unit 1)
 		(exclude_from_sim no)
 		(in_bom yes)
-		(on_board yes)
+		(on_board no)
 		(dnp no)
 		(fields_autoplaced yes)
 		(property "Reference" "U13"
-			(at 154.94 45.72 0)
+			(at 104.14 58.42 0)
 			(effects
 				(font
@@
 		)
 		(property "Value" "Teensy4.1"
-			(at 154.94 48.26 0)
+			(at 104.14 60.96 0)
 			(effects
 				(font
@@
 		)
 		(property "Footprint" ""
-			(at 144.78 101.6 0)
+			(at 93.98 114.3 0)
 			(effects
 				(font
@@
 		)
 		(property "Datasheet" ""
-			(at 144.78 101.6 0)
+			(at 93.98 114.3 0)
 			(effects
 				(font
@@
 		)
 		(property "Description" ""
-			(at 154.94 111.76 0)
-			(effects
-				(font
+			(at 104.14 124.46 0)
+			(effects
+				(font
+					(size 1.27 1.27)
+				)
+				(hide yes)
+			)
+		)
+		(property "Purchase Link" ""
+			(at 104.14 124.46 0)
+			(effects
+				(font

Commit message: Save progress
Connections:
- net GND: now reaches J_Teensy_Right.10 (Pin_10)
- net GND: now also J_Teensy_Left.1 (Pin_1), J_Teensy_Right.23 (Pin_23)
- net 3.3V: now reaches J_Teensy_Right.22 (Pin_22)
- net 3.3V: now also J_Teensy_Left.15 (Pin_15)
Changed lines of the file:
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@@
 		(at 76.2 135.89)
 	)
+	(hierarchical_label "GND"
+		(shape bidirectional)
+		(at 157.48 105.41 0)
+		(effects
+			(font
+				(size 1.27 1.27)
+			)
+			(justify left)
+		)
+	)
+	(hierarchical_label "GND"
+		(shape bidirectional)
+		(at 157.48 72.39 0)
+		(effects
+			(font
+				(size 1.27 1.27)
+			)
+			(justify left)
+		)
+	)
 	(hierarchical_label "CS_DAC"
 		(shape output)
@@
 		)
 	)
+	(hierarchical_label "GND"
+		(shape bidirectional)
+		(at 50.8 69.85 180)
+		(effects
+			(font
+				(size 1.27 1.27)
+			)
+			(justify right)
+		)
+	)
+	(hierarchical_label "3.3V"
+		(shape output)
+		(at 50.8 105.41 180)
+		(effects
+			(font
+				(size 1.27 1.27)
+			)
+			(justify right)
+		)
+	)
 	(hierarchical_label "SCK"
 		(shape output)
@@
 			)
 			(justify right)
+		)
+	)
+	(hierarchical_label "3.3V"
+		(shape output)
+		(at 157.48 74.93 0)
+		(effects
+			(font
+				(size 1.27 1.27)
+			)
+			(justify left)
 		)
 	)
@@
 		(dnp no)
 		(property "Reference" "J_Teensy_Right"
-			(at 158.75 61.468 0)
+			(at 159.512 62.992 0)
 			(effects
 				(font
@@
 		)
 		(property "Value" "Conn_01x24_Socket"
-			(at 161.29 64.262 0)
+			(at 162.052 65.786 0)
 			(effects
 				(font
@@
 		(dnp no)
 		(property "Reference" "J11"
-			(at 134.366 62.992 0)
+			(at 134.112 63.246 0)
 			(effects
 				(font
@@
 		)
 		(property "Value" "Conn_01x24_Pin"
-			(at 134.366 65.532 0)
-			(effects
-				(font
+			(at 134.112 65.786 0)
+			(effects
+				(font
