File: Models/TransimpedanceAmplifier/TIA_OneStage.kicad_sch (KiCad schematic)
At the start: 7 parts, among them J5 Conn_01x02_Pin, J6 Conn_01x02_Pin, U4 OPA828ID

Commit message: Save progress
Parts:
- U4: footprint D8_TEX -> (none)
Changed lines of the file:
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@@
 			)
 		)
-		(property "Footprint" "D8_TEX"
+		(property "Footprint" ""
 			(at 78.74 93.98 0)
 			(effects

Commit message: Save progress
Parts:
- U4: value OPA828ID -> OPA828
Changed lines of the file:
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@@
 			)
 		)
-		(property "Value" "OPA828ID"
+		(property "Value" "OPA828"
 			(at 99.06 86.36 0)
 			(effects
