File: Models/TransimpedanceAmplifier/CPU.kicad_sch (KiCad schematic)
At the start: 0 parts

Commit message: Save progress
Other:
- sheet Isolation ports: added 3.3V_Analog, 3.3V_Digital, CS_ADC_Analog, CS_ADC_Digital, CS_DAC_Analog, CS_DAC_Digital, GND_Analog, GND_Digital, MISO_ADC_Analog, MISO_DAC_Analog, MISO_Digital, MOSI_ADC_Analog, MOSI_DAC_Analog, MOSI_Digital, SCK_ADC_Analog, SCK_DAC_Analog, SCK_Digital; removed none
- sheet Teensy ports: added CS_ADC, CS_DAC, MISO, MOSI, SCK; removed none

Commit message: Save progress after a major refactoring
Other:
- added sheet ADC (ADC.kicad_sch)
- added sheet DAC (DAC.kicad_sch)

Commit message: Save progress
Other:
- sheet Teensy ports: added 3.3V, GND; removed none
Changed lines of the file:
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@@
+	(wire
+		(pts
+			(xy 60.96 35.56) (xy 76.2 35.56)
+		)
+		(stroke
+			(width 0)
+			(type default)
+		)
+	)
 	(wire
 		(pts
@@
 		(pts
 			(xy 152.4 35.56) (xy 157.48 35.56)
+		)
+		(stroke
+			(width 0)
+			(type default)
+		)
+	)
+	(wire
+		(pts
+			(xy 60.96 30.48) (xy 76.2 30.48)
 		)
 		(stroke
@@
 			(effects
 				(font
+					(size 1.27 1.27)
+				)
+				(justify right)
+			)
+		)
+		(pin "3.3V" output
+			(at 60.96 30.48 0)
+			(effects
+				(font
+					(size 1.27 1.27)
+				)
+				(justify right)
+			)
+		)
+		(pin "GND" bidirectional
+			(at 60.96 35.56 0)
+			(effects
+				(font
