File: Models/TransimpedanceAmplifier/HighVoltage.kicad_sch (KiCad schematic)
At the start: 8 parts, among them U6 LM7915, -15V, 5%, U7 LM7815, 15V, 5%

Commit message: Starting major changes in response to the SOIC-8 version of OP37 being out of stock
Parts:
- U6: Cost $0.00 -> $1.48; Cost (qty10) (none) -> $1.079; RoHS Compliant NO -> YES
- U7: Cost $0.00 -> $1.80; Cost (qty10) (none) -> $1.325; RoHS Compliant NO -> YES
Changed lines of the file:
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@@
 			)
 		)
-		(property "Cost" "$0.00"
+		(property "Cost" "$1.48"
 			(at 53.34 132.08 0)
 			(effects
@@
 			)
 		)
-		(property "RoHS Compliant" "NO"
+		(property "RoHS Compliant" "YES"
+			(at 53.34 132.08 0)
+			(effects
+				(font
+					(size 1.27 1.27)
+				)
+				(hide yes)
+			)
+		)
+		(property "Cost (qty10)" "$1.079"
 			(at 53.34 132.08 0)
 			(effects
@@
 			)
 		)
-		(property "Cost" "$0.00"
-			(at 58.42 55.88 0)
-			(effects
-				(font
-					(size 1.27 1.27)
-				)
-				(hide yes)
-			)
-		)
-		(property "RoHS Compliant" "NO"
-			(at 58.42 55.88 0)
-			(effects
+		(property "Cost" "$1.80"
+			(at 58.42 55.88 0)
+			(effects
+				(font
+					(size 1.27 1.27)
+				)
+				(hide yes)
+			)
+		)
+		(property "RoHS Compliant" "YES"
+			(at 58.42 55.88 0)
+			(effects
+				(font
+					(size 1.27 1.27)
+				)
+				(hide yes)
+			)
+		)
+		(property "Cost (qty10)" "$1.325"
+			(at 58.42 55.88 0)
+			(effects
