File: Models/TransimpedanceAmplifier/LowVoltage_Converter.kicad_sch (KiCad schematic)
At the start: 8 parts, among them U8 LM7805, 5V, 5%, U9 TLV76133, 3.3V, 1%

Commit message: Working on filling in the last details of the schematics
Parts:
- C21, C23: footprint (none) -> TwoTerminal:CAPC0603; Cost (none) -> $0.00; RoHS Compliant (none) -> NO
- C22, C24: footprint (none) -> TwoTerminal:CAPC0805; Cost (none) -> $0.00; RoHS Compliant (none) -> NO
- D10, D11: footprint (none) -> TwoTerminal:SOD-123; Cost (none) -> $0.00; RoHS Compliant (none) -> NO
- U8, U9: Cost (none) -> $0.00; RoHS Compliant (none) -> NO
Changed lines of the file:
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@@
 			)
 		)
-		(property "Footprint" ""
+		(property "Footprint" "TwoTerminal:CAPC0805"
 			(at 115.2652 147.32 0)
 			(effects
@@
 			)
 		)
+		(property "Cost" "$0.00"
+			(at 114.3 143.51 0)
+			(effects
+				(font
+					(size 1.27 1.27)
+				)
+				(hide yes)
+			)
+		)
+		(property "RoHS Compliant" "NO"
+			(at 114.3 143.51 0)
+			(effects
+				(font
+					(size 1.27 1.27)
+				)
+				(hide yes)
+			)
+		)
 		(pin "1"
 		)
@@
 		)
 		(property "Purchase Link" "https://www.digikey.com/en/products/detail/texas-instruments/LM7805CT-NOPB/3901929"
+			(at 58.42 55.88 0)
+			(effects
+				(font
+					(size 1.27 1.27)
+				)
+				(hide yes)
+			)
+		)
+		(property "Cost" "$0.00"
+			(at 58.42 55.88 0)
+			(effects
+				(font
+					(size 1.27 1.27)
+				)
+				(hide yes)
+			)
+		)
+		(property "RoHS Compliant" "NO"
 			(at 58.42 55.88 0)
 			(effects
@@
 			)
 		)
-		(property "Footprint" ""
+		(property "Footprint" "TwoTerminal:SOD-123"
 			(at 134.62 64.77 0)
 			(effects
@@
 			)
 		)
+		(property "Cost" "$0.00"
+			(at 134.62 64.77 90)
+			(effects
+				(font
+					(size 1.27 1.27)
+				)
+				(hide yes)
+			)
+		)
+		(property "RoHS Compliant" "NO"
+			(at 134.62 64.77 90)
+			(effects
+				(font
+					(size 1.27 1.27)
+				)
+				(hide yes)
+			)
+		)
 		(pin "1"
 		)
@@
 			)
 		)
-		(property "Footprint" ""
+		(property "Footprint" "TwoTerminal:CAPC0805"
 			(at 72.0852 152.4 0)
 			(effects
@@
 			)
 		)
+		(property "Cost" "$0.00"
+			(at 71.12 148.59 0)
+			(effects
+				(font
+					(size 1.27 1.27)
+				)
+				(hide yes)
+			)
+		)
+		(property "RoHS Compliant" "NO"
+			(at 71.12 148.59 0)
+			(effects
+				(font
+					(size 1.27 1.27)
+				)
+				(hide yes)
+			)
+		)
 		(pin "1"
 		)
@@
 			)
 		)
-		(property "Footprint" ""
+		(property "Footprint" "TwoTerminal:CAPC0603"
 			(at 54.3052 71.12 0)
 			(effects
@@
 			)
 		)
+		(property "Cost" "$0.00"
+			(at 53.34 67.31 0)
+			(effects
+				(font
+					(size 1.27 1.27)
+				)
+				(hide yes)
+			)
+		)
+		(property "RoHS Compliant" "NO"
+			(at 53.34 67.31 0)
+			(effects
+				(font
+					(size 1.27 1.27)
+				)
+				(hide yes)
+			)
+		)
 		(pin "2"
 		)
@@
 			)
 		)
-		(property "Footprint" ""
+		(property "Footprint" "TwoTerminal:SOD-123"
 			(at 134.62 143.51 0)
 			(effects
@@
 			)
 		)
+		(property "Cost" "$0.00"
+			(at 134.62 143.51 90)
+			(effects
+				(font
+					(size 1.27 1.27)
+				)
+				(hide yes)
+			)
+		)
+		(property "RoHS Compliant" "NO"
+			(at 134.62 143.51 90)
+			(effects
+				(font
+					(size 1.27 1.27)
+				)
+				(hide yes)
+			)
+		)
 		(pin "1"
 		)
@@
 			)
 		)
-		(property "Footprint" ""
+		(property "Footprint" "TwoTerminal:CAPC0603"
 			(at 112.7252 68.58 0)
 			(effects
@@
 			)
 		)
+		(property "Cost" "$0.00"
+			(at 111.76 64.77 0)
+			(effects
+				(font
+					(size 1.27 1.27)
+				)
+				(hide yes)
+			)
+		)
+		(property "RoHS Compliant" "NO"
+			(at 111.76 64.77 0)
+			(effects
+				(font
+					(size 1.27 1.27)
+				)
+				(hide yes)
+			)
+		)
 		(pin "1"
 		)
@@
 			(at 77.47 130.81 0)
 			(effects
+				(font
+					(size 1.27 1.27)
+				)
+				(hide yes)
+			)
+		)
+		(property "Cost" "$0.00"
+			(at 77.47 130.81 0)
+			(effects
+				(font
+					(size 1.27 1.27)
+				)
+				(hide yes)
+			)
+		)
+		(property "RoHS Compliant" "NO"
+			(at 77.47 130.81 0)
+			(effects

Commit message: Fixed a bug in footprint assignment
Parts:
- U8: footprint (none) -> ThreeTerminal:TO-220
- U9: footprint (none) -> ThreeTerminal:SOT-223
Changed lines of the file:
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@@
 			)
 		)
-		(property "Footprint" ""
+		(property "Footprint" "ThreeTerminal:TO-220"
 			(at 58.42 55.88 0)
 			(effects
@@
 			)
 		)
-		(property "Footprint" ""
+		(property "Footprint" "ThreeTerminal:SOT-223"
 			(at 77.47 130.81 0)
 			(effects

Commit message: Save progress
Parts:
- C21: Cost $0.00 -> $0.14; Cost (qty10) (none) -> $0.078; RoHS Compliant NO -> YES
- C22, C24: Cost $0.00 -> $0.21; Cost (qty10) (none) -> $0.121; RoHS Compliant NO -> YES
- C23: Cost $0.00 -> $0.15; Cost (qty10) (none) -> $0.087; RoHS Compliant NO -> YES
- D10, D11: Cost $0.00 -> $0.34; Cost (qty10) (none) -> $0.220; RoHS Compliant NO -> YES
Changed lines of the file:
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@@
 			)
 		)
-		(property "Cost" "$0.00"
+		(property "Cost" "$0.21"
 			(at 114.3 143.51 0)
 			(effects
@@
 			)
 		)
-		(property "RoHS Compliant" "NO"
+		(property "RoHS Compliant" "YES"
+			(at 114.3 143.51 0)
+			(effects
+				(font
+					(size 1.27 1.27)
+				)
+				(hide yes)
+			)
+		)
+		(property "Cost (qty10)" "$0.121"
 			(at 114.3 143.51 0)
 			(effects
@@
 			)
 		)
-		(property "Cost" "$0.00"
+		(property "Cost" "$0.34"
 			(at 134.62 64.77 90)
 			(effects
@@
 			)
 		)
-		(property "RoHS Compliant" "NO"
+		(property "RoHS Compliant" "YES"
+			(at 134.62 64.77 90)
+			(effects
+				(font
+					(size 1.27 1.27)
+				)
+				(hide yes)
+			)
+		)
+		(property "Cost (qty10)" "$0.220"
 			(at 134.62 64.77 90)
 			(effects
@@
 			)
 		)
-		(property "Cost" "$0.00"
+		(property "Cost" "$0.21"
 			(at 71.12 148.59 0)
 			(effects
@@
 			)
 		)
-		(property "RoHS Compliant" "NO"
+		(property "RoHS Compliant" "YES"
+			(at 71.12 148.59 0)
+			(effects
+				(font
+					(size 1.27 1.27)
+				)
+				(hide yes)
+			)
+		)
+		(property "Cost (qty10)" "$0.121"
 			(at 71.12 148.59 0)
 			(effects
@@
 			)
 		)
-		(property "Cost" "$0.00"
+		(property "Cost" "$0.14"
 			(at 53.34 67.31 0)
 			(effects
@@
 			)
 		)
-		(property "RoHS Compliant" "NO"
+		(property "RoHS Compliant" "YES"
+			(at 53.34 67.31 0)
+			(effects
+				(font
+					(size 1.27 1.27)
+				)
+				(hide yes)
+			)
+		)
+		(property "Cost (qty10)" "$0.078"
 			(at 53.34 67.31 0)
 			(effects
@@
 			)
 		)
-		(property "Cost" "$0.00"
+		(property "Cost" "$0.34"
 			(at 134.62 143.51 90)
 			(effects
@@
 			)
 		)
-		(property "RoHS Compliant" "NO"
+		(property "RoHS Compliant" "YES"
+			(at 134.62 143.51 90)
+			(effects
+				(font
+					(size 1.27 1.27)
+				)
+				(hide yes)
+			)
+		)
+		(property "Cost (qty10)" "$0.220"
 			(at 134.62 143.51 90)
 			(effects
@@
 			)
 		)
-		(property "Cost" "$0.00"
+		(property "Cost" "$0.15"
 			(at 111.76 64.77 0)
 			(effects
@@
 			)
 		)
-		(property "RoHS Compliant" "NO"
+		(property "RoHS Compliant" "YES"
 			(at 111.76 64.77 0)
 			(effects
+				(font
+					(size 1.27 1.27)
+				)
+				(hide yes)
+			)
+		)
+		(property "Cost (qty10)" "$0.087"
+			(at 111.76 64.77 0)
+			(effects
