File: Models/TransimpedanceAmplifier/LowVoltage_Converter.kicad_sch (KiCad schematic)
At the start: 8 parts, among them U8 LM7805, 5V, 5%, U9 TLV76133, 3.3V, 1%

Commit message: Going to shift all the expensive, hard-to-find ICs over to Mouser
Parts:
- U8: Cost $0.00 -> $1.80; Cost (qty10) (none) -> $1.325; RoHS Compliant NO -> YES
Changed lines of the file:
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@@
 			)
 		)
-		(property "Cost" "$0.00"
+		(property "Cost" "$1.80"
 			(at 58.42 55.88 0)
 			(effects
@@
 			)
 		)
-		(property "RoHS Compliant" "NO"
+		(property "RoHS Compliant" "YES"
 			(at 58.42 55.88 0)
 			(effects
+				(font
+					(size 1.27 1.27)
+				)
+				(hide yes)
+			)
+		)
+		(property "Cost (qty10)" "$1.325"
+			(at 58.42 55.88 0)
+			(effects

Commit message: Starting major changes in response to the SOIC-8 version of OP37 being out of stock
Parts:
- U9: Cost $0.00 -> $0.48; Cost (qty10) (none) -> $0.33; RoHS Compliant NO -> YES
Changed lines of the file:
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@@
 			)
 		)
-		(property "Cost" "$0.00"
+		(property "Cost" "$0.48"
 			(at 77.47 130.81 0)
 			(effects
@@
 			)
 		)
-		(property "RoHS Compliant" "NO"
+		(property "RoHS Compliant" "YES"
 			(at 77.47 130.81 0)
 			(effects
+				(font
+					(size 1.27 1.27)
+				)
+				(hide yes)
+			)
+		)
+		(property "Cost (qty10)" "$0.33"
+			(at 77.47 130.81 0)
+			(effects
