File: Models/TransimpedanceAmplifier/TransimpedanceAmplifier.kicad_sch (KiCad schematic)
At the start: 4 parts, among them J1 Conn_01x02_Socket, J2 Conn_01x02_Socket, J3 Conn_01x03_Pin

Commit message: Fixed a bug in footprint assignment
Parts:
- R1: footprint (none) -> TwoTerminal:RESC0603
Changed lines of the file:
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@@
 			)
 		)
-		(property "Footprint" ""
+		(property "Footprint" "TwoTerminal:RESC0603"
 			(at 41.656 54.864 90)
 			(effects

Commit message: Save progress
Parts:
- J1, J2: Cost $0.00 -> $0.24; Cost (qty10) (none) -> $0.206; RoHS Compliant NO -> YES
- J3: Cost $0.00 -> $0.10; Cost (qty10) (none) -> $0.025; RoHS Compliant NO -> YES
Changed lines of the file:
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@@
 			)
 		)
-		(property "Cost" "$0.00"
+		(property "Cost" "$0.24"
 			(at 93.98 123.19 0)
 			(effects
@@
 			)
 		)
-		(property "RoHS Compliant" "NO"
+		(property "RoHS Compliant" "YES"
+			(at 93.98 123.19 0)
+			(effects
+				(font
+					(size 1.27 1.27)
+				)
+				(hide yes)
+			)
+		)
+		(property "Cost (qty10)" "$0.206"
 			(at 93.98 123.19 0)
 			(effects
@@
 			)
 		)
-		(property "Cost" "$0.00"
-			(at 160.02 121.92 0)
-			(effects
-				(font
-					(size 1.27 1.27)
-				)
-				(hide yes)
-			)
-		)
-		(property "RoHS Compliant" "NO"
+		(property "Cost" "$0.10"
+			(at 160.02 121.92 0)
+			(effects
+				(font
+					(size 1.27 1.27)
+				)
+				(hide yes)
+			)
+		)
+		(property "RoHS Compliant" "YES"
+			(at 160.02 121.92 0)
+			(effects
+				(font
+					(size 1.27 1.27)
+				)
+				(hide yes)
+			)
+		)
+		(property "Cost (qty10)" "$0.025"
 			(at 160.02 121.92 0)
 			(effects
@@
 			)
 		)
-		(property "Cost" "$0.00"
+		(property "Cost" "$0.24"
 			(at 45.72 116.84 90)
 			(effects
@@
 			)
 		)
-		(property "RoHS Compliant" "NO"
+		(property "RoHS Compliant" "YES"
 			(at 45.72 116.84 90)
 			(effects
+				(font
+					(size 1.27 1.27)
+				)
+				(hide yes)
+			)
+		)
+		(property "Cost (qty10)" "$0.206"
+			(at 45.72 116.84 90)
+			(effects

Commit message: Added important links regarding high-voltage electronics
Parts:
- R1: Cost $0.00 -> $0.10; Cost (qty10) (none) -> $0.030; RoHS Compliant NO -> YES
Changed lines of the file:
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@@
 			)
 		)
-		(property "Cost" "$0.00"
+		(property "Cost" "$0.10"
 			(at 40.64 54.61 0)
 			(effects
@@
 			)
 		)
-		(property "RoHS Compliant" "NO"
+		(property "RoHS Compliant" "YES"
 			(at 40.64 54.61 0)
 			(effects
+				(font
+					(size 1.27 1.27)
+				)
+				(hide yes)
+			)
+		)
+		(property "Cost (qty10)" "$0.030"
+			(at 40.64 54.61 0)
+			(effects
