File: Models/TransimpedanceAmplifier/PreAmplifier.kicad_sch (KiCad schematic)
At the start: 12 parts, among them J14 Conn_01x02_Pin, J15 Conn_01x02_Pin, U4 AD8615

Commit message: Completely fixed the batteries
Parts:
- renumbered J14 to J6, J15 to J7
Changed lines of the file:
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@@
 		(dnp no)
 		(fields_autoplaced yes)
-		(property "Reference" "J15"
+		(property "Reference" "J7"
 			(at 247.65 35.5599 0)
 			(effects
@@
 			(project ""
 				(path "/ec9f2ae3-e40d-40eb-9760-2b611ee8efd1/226b3d0c-9e45-4bcf-9bef-58938aee743e/728283d1-1c30-4fdc-aa4d-bf897972ea87"
-					(reference "J15")
+					(reference "J7")
 					(unit 1)
 				)
@@
 		(dnp no)
 		(fields_autoplaced yes)
-		(property "Reference" "J14"
+		(property "Reference" "J6"
 			(at 227.33 139.6999 0)
 			(effects
@@
 			(project "TransimpedanceAmplifier"
 				(path "/ec9f2ae3-e40d-40eb-9760-2b611ee8efd1/226b3d0c-9e45-4bcf-9bef-58938aee743e/728283d1-1c30-4fdc-aa4d-bf897972ea87"
-					(reference "J14")
+					(reference "J6")
 					(unit 1)
 				)

Commit message: Finalized the last detail of the schematic
Parts:
- renumbered R9 to R10, R10 to R11, R7 to R8, R8 to R9
Changed lines of the file:
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@@
 	(text "TODO: (1 kΩ trimpot)\nFlip the polarity of pins 1 and 3\nbased on which is more convenient for the\nphysical layout on the PCB"
 		(exclude_from_sim no)
-		(at 186.182 25.908 0)
+		(at 185.928 21.844 0)
 		(effects
 			(font
@@
 		(dnp no)
 		(fields_autoplaced yes)
-		(property "Reference" "R7"
+		(property "Reference" "R8"
 			(at 223.52 58.4199 0)
 			(effects
@@
 			(project ""
 				(path "/ec9f2ae3-e40d-40eb-9760-2b611ee8efd1/226b3d0c-9e45-4bcf-9bef-58938aee743e/728283d1-1c30-4fdc-aa4d-bf897972ea87"
-					(reference "R7")
+					(reference "R8")
 					(unit 1)
 				)
@@
 		(on_board yes)
 		(dnp no)
-		(property "Reference" "R10"
+		(property "Reference" "R11"
 			(at 243.84 52.0699 0)
 			(effects
@@
 			(project ""
 				(path "/ec9f2ae3-e40d-40eb-9760-2b611ee8efd1/226b3d0c-9e45-4bcf-9bef-58938aee743e/728283d1-1c30-4fdc-aa4d-bf897972ea87"
-					(reference "R10")
+					(reference "R11")
 					(unit 1)
 				)
@@
 		(dnp no)
 		(fields_autoplaced yes)
-		(property "Reference" "R8"
+		(property "Reference" "R9"
 			(at 223.52 106.6799 0)
 			(effects
@@
 			(project ""
 				(path "/ec9f2ae3-e40d-40eb-9760-2b611ee8efd1/226b3d0c-9e45-4bcf-9bef-58938aee743e/728283d1-1c30-4fdc-aa4d-bf897972ea87"
-					(reference "R8")
+					(reference "R9")
 					(unit 1)
 				)
@@
 		(dnp no)
 		(fields_autoplaced yes)
-		(property "Reference" "R9"
+		(property "Reference" "R10"
 			(at 223.52 119.3799 0)
 			(effects
@@
 			(project ""
 				(path "/ec9f2ae3-e40d-40eb-9760-2b611ee8efd1/226b3d0c-9e45-4bcf-9bef-58938aee743e/728283d1-1c30-4fdc-aa4d-bf897972ea87"
-					(reference "R9")
+					(reference "R10")
 					(unit 1)
 				)

Commit message: Working on filling in the last details of the schematics
Parts:
- C11, C12: footprint (none) -> TwoTerminal:CAPC0603; Cost (none) -> $0.00; RoHS Compliant (none) -> NO
- C13, C14: footprint (none) -> TwoTerminal:CAPC0805; Cost (none) -> $0.00; RoHS Compliant (none) -> NO
- D3: footprint (none) -> ThreeTerminal:SOT-23; Cost (none) -> $0.00; RoHS Compliant (none) -> NO
- J6, J7: footprint (none) -> Connector_Custom:PinHeader_1x2; Cost (none) -> $0.00; RoHS Compliant (none) -> NO
- R10, R11, R8, R9, U4: Cost (none) -> $0.00; RoHS Compliant (none) -> NO
Other:
- note added: "NO"
Changed lines of the file:
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@@
+		)
+	)
+	(text "NO"
+		(exclude_from_sim no)
+		(at 93.98 124.46 0)
+		(effects
+			(font
+				(size 1.27 1.27)
+			)
 		)
 	)
@@
 			)
 		)
+		(property "Cost" "$0.00"
+			(at 220.98 59.69 0)
+			(effects
+				(font
+					(size 1.27 1.27)
+				)
+				(hide yes)
+			)
+		)
+		(property "RoHS Compliant" "NO"
+			(at 220.98 59.69 0)
+			(effects
+				(font
+					(size 1.27 1.27)
+				)
+				(hide yes)
+			)
+		)
 		(pin "2"
 		)
@@
 			)
 		)
-		(property "Footprint" ""
+		(property "Footprint" "ThreeTerminal:SOT-23"
 			(at 220.98 80.01 0)
 			(effects
@@
 		)
 		(property "Purchase Link" "https://www.digikey.com/en/products/detail/diodes-incorporated/LM4040D33FTA/10295608"
+			(at 220.98 80.01 0)
+			(effects
+				(font
+					(size 1.27 1.27)
+				)
+				(hide yes)
+			)
+		)
+		(property "Cost" "$0.00"
+			(at 220.98 80.01 0)
+			(effects
+				(font
+					(size 1.27 1.27)
+				)
+				(hide yes)
+			)
+		)
+		(property "RoHS Compliant" "NO"
 			(at 220.98 80.01 0)
 			(effects
@@
 		)
 		(property "Purchase Link" "https://www.digikey.com/en/products/detail/bourns-inc/3296Y-1-102LF/1088084"
+			(at 241.3 53.34 0)
+			(effects
+				(font
+					(size 1.27 1.27)
+				)
+				(hide yes)
+			)
+		)
+		(property "Cost" "$0.00"
+			(at 241.3 53.34 0)
+			(effects
+				(font
+					(size 1.27 1.27)
+				)
+				(hide yes)
+			)
+		)
+		(property "RoHS Compliant" "NO"
 			(at 241.3 53.34 0)
 			(effects
@@
 			)
 		)
+		(property "Cost" "$0.00"
+			(at 220.98 107.95 0)
+			(effects
+				(font
+					(size 1.27 1.27)
+				)
+				(hide yes)
+			)
+		)
+		(property "RoHS Compliant" "NO"
+			(at 220.98 107.95 0)
+			(effects
+				(font
+					(size 1.27 1.27)
+				)
+				(hide yes)
+			)
+		)
 		(pin "1"
 		)
@@
 			)
 		)
-		(property "Footprint" ""
+		(property "Footprint" "TwoTerminal:CAPC0603"
 			(at 160.9852 87.63 0)
 			(effects
@@
 		)
 		(property "Purchase Link" "https://www.digikey.com/en/products/detail/murata-electronics/GRT188R61H105KE13D/5416752"
+			(at 160.02 83.82 0)
+			(effects
+				(font
+					(size 1.27 1.27)
+				)
+				(hide yes)
+			)
+		)
+		(property "Cost" "$0.00"
+			(at 160.02 83.82 0)
+			(effects
+				(font
+					(size 1.27 1.27)
+				)
+				(hide yes)
+			)
+		)
+		(property "RoHS Compliant" "NO"
 			(at 160.02 83.82 0)
 			(effects
@@
 			)
 		)
-		(property "Footprint" ""
+		(property "Footprint" "TwoTerminal:CAPC0603"
 			(at 160.9852 116.84 0)
 			(effects
@@
 		)
 		(property "Purchase Link" "https://www.digikey.com/en/products/detail/murata-electronics/GRT188R61H105KE13D/5416752"
+			(at 160.02 113.03 0)
+			(effects
+				(font
+					(size 1.27 1.27)
+				)
+				(hide yes)
+			)
+		)
+		(property "Cost" "$0.00"
+			(at 160.02 113.03 0)
+			(effects
+				(font
+					(size 1.27 1.27)
+				)
+				(hide yes)
+			)
+		)
+		(property "RoHS Compliant" "NO"
 			(at 160.02 113.03 0)
 			(effects
@@
 			)
 		)
-		(property "Footprint" ""
+		(property "Footprint" "TwoTerminal:CAPC0805"
 			(at 181.3052 87.63 0)
 			(effects
@@
 		)
 		(property "Purchase Link" "https://www.digikey.com/en/products/detail/murata-electronics/GRM21BR61E106KA73K/4905532"
+			(at 180.34 83.82 0)
+			(effects
+				(font
+					(size 1.27 1.27)
+				)
+				(hide yes)
+			)
+		)
+		(property "Cost" "$0.00"
+			(at 180.34 83.82 0)
+			(effects
+				(font
+					(size 1.27 1.27)
+				)
+				(hide yes)
+			)
+		)
+		(property "RoHS Compliant" "NO"
 			(at 180.34 83.82 0)
 			(effects
@@
 			)
 		)
-		(property "Footprint" ""
+		(property "Footprint" "Connector_Custom:PinHeader_1x2"
 			(at 246.38 38.1 0)
 			(effects
@@
 		)
 		(property "Purchase Link" "https://www.digikey.com/en/products/detail/sullins-connector-solutions/QPC02SXGN-RC/2618262"
+			(at 246.38 38.1 0)
+			(effects
+				(font
+					(size 1.27 1.27)
+				)
+				(hide yes)
+			)
+		)
+		(property "Cost" "$0.00"
+			(at 246.38 38.1 0)
+			(effects
+				(font
+					(size 1.27 1.27)
+				)
+				(hide yes)
+			)
+		)
+		(property "RoHS Compliant" "NO"
 			(at 246.38 38.1 0)
 			(effects
@@
 			)
 		)
+		(property "Cost" "$0.00"
+			(at 220.98 120.65 0)
+			(effects
+				(font
+					(size 1.27 1.27)
+				)
+				(hide yes)
+			)
+		)
+		(property "RoHS Compliant" "NO"
+			(at 220.98 120.65 0)
+			(effects
+				(font
+					(size 1.27 1.27)
+				)
+				(hide yes)
+			)
+		)
 		(pin "1"
 		)
@@
 			)
 		)
-		(property "Footprint" ""
+		(property "Footprint" "Connector_Custom:PinHeader_1x2"
 			(at 226.06 142.24 0)
 			(effects
@@
 		)
 		(property "Purchase Link" "https://www.digikey.com/en/products/detail/sullins-connector-solutions/QPC02SXGN-RC/2618262"
+			(at 226.06 142.24 0)
+			(effects
+				(font
+					(size 1.27 1.27)
+				)
+				(hide yes)
+			)
+		)
+		(property "Cost" "$0.00"
+			(at 226.06 142.24 0)
+			(effects
+				(font
+					(size 1.27 1.27)
+				)
+				(hide yes)
+			)
+		)
+		(property "RoHS Compliant" "NO"
 			(at 226.06 142.24 0)
 			(effects
@@
 			)
 		)
-		(property "Footprint" ""
+		(property "Footprint" "TwoTerminal:CAPC0805"
 			(at 181.3052 116.84 0)
 			(effects
@@
 		)
 		(property "Purchase Link" "https://www.digikey.com/en/products/detail/murata-electronics/GRM21BR61E106KA73K/4905532"
+			(at 180.34 113.03 0)
+			(effects
+				(font
+					(size 1.27 1.27)
+				)
+				(hide yes)
+			)
+		)
+		(property "Cost" "$0.00"
+			(at 180.34 113.03 0)
+			(effects
+				(font
+					(size 1.27 1.27)
+				)
+				(hide yes)
+			)
+		)
+		(property "RoHS Compliant" "NO"
 			(at 180.34 113.03 0)
 			(effects
@@
 			(at 43.18 81.28 0)
 			(effects
+				(font
+					(size 1.27 1.27)
+				)
+				(hide yes)
+			)
+		)
+		(property "Cost" "$0.00"
+			(at 43.18 81.28 0)
+			(effects
+				(font
+					(size 1.27 1.27)
+				)
+				(hide yes)
+			)
+		)
+		(property "RoHS Compliant" "NO"
+			(at 43.18 81.28 0)
+			(effects

Commit message: Fixed a bug in footprint assignment
Parts:
- R10, R8, R9: footprint (none) -> TwoTerminal:RESC0603
- R11: footprint (none) -> ThreeTerminal:Bourns_3296Y
- U4: footprint (none) -> IC:AD8615
Changed lines of the file:
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@@
 			)
 		)
-		(property "Footprint" ""
+		(property "Footprint" "TwoTerminal:RESC0603"
 			(at 221.996 59.944 90)
 			(effects
@@
 			)
 		)
-		(property "Footprint" ""
+		(property "Footprint" "ThreeTerminal:Bourns_3296Y"
 			(at 241.3 53.34 0)
 			(effects
@@
 			)
 		)
-		(property "Footprint" ""
+		(property "Footprint" "TwoTerminal:RESC0603"
 			(at 221.996 108.204 90)
 			(effects
@@
 			)
 		)
-		(property "Footprint" ""
+		(property "Footprint" "TwoTerminal:RESC0603"
 			(at 221.996 120.904 90)
 			(effects
@@
 			)
 		)
-		(property "Footprint" ""
+		(property "Footprint" "IC:AD8615"
 			(at 43.18 81.28 0)
 			(effects

Commit message: Save progress
Parts:
- C11, C12: Cost $0.00 -> $0.14; Cost (qty10) (none) -> $0.078; RoHS Compliant NO -> YES
- C13, C14: Cost $0.00 -> $0.16; Cost (qty10) (none) -> $0.090; RoHS Compliant NO -> YES
- D3: Cost $0.00 -> $0.36; Cost (qty10) (none) -> $0.250; RoHS Compliant NO -> YES
- J6, J7: Cost $0.00 -> $0.10; Cost (qty10) (none) -> $0.025; RoHS Compliant NO -> YES
Changed lines of the file:
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@@
 			)
 		)
-		(property "Cost" "$0.00"
+		(property "Cost" "$0.36"
 			(at 220.98 80.01 0)
 			(effects
@@
 			)
 		)
-		(property "RoHS Compliant" "NO"
+		(property "RoHS Compliant" "YES"
+			(at 220.98 80.01 0)
+			(effects
+				(font
+					(size 1.27 1.27)
+				)
+				(hide yes)
+			)
+		)
+		(property "Cost (qty10)" "$0.250"
 			(at 220.98 80.01 0)
 			(effects
@@
 			)
 		)
-		(property "Cost" "$0.00"
+		(property "Cost" "$0.14"
 			(at 160.02 83.82 0)
 			(effects
@@
 			)
 		)
-		(property "RoHS Compliant" "NO"
+		(property "RoHS Compliant" "YES"
+			(at 160.02 83.82 0)
+			(effects
+				(font
+					(size 1.27 1.27)
+				)
+				(hide yes)
+			)
+		)
+		(property "Cost (qty10)" "$0.078"
 			(at 160.02 83.82 0)
 			(effects
@@
 			)
 		)
-		(property "Cost" "$0.00"
+		(property "Cost" "$0.14"
 			(at 160.02 113.03 0)
 			(effects
@@
 			)
 		)
-		(property "RoHS Compliant" "NO"
+		(property "RoHS Compliant" "YES"
+			(at 160.02 113.03 0)
+			(effects
+				(font
+					(size 1.27 1.27)
+				)
+				(hide yes)
+			)
+		)
+		(property "Cost (qty10)" "$0.078"
 			(at 160.02 113.03 0)
 			(effects
@@
 			)
 		)
-		(property "Cost" "$0.00"
+		(property "Cost" "$0.16"
 			(at 180.34 83.82 0)
 			(effects
@@
 			)
 		)
-		(property "RoHS Compliant" "NO"
+		(property "RoHS Compliant" "YES"
+			(at 180.34 83.82 0)
+			(effects
+				(font
+					(size 1.27 1.27)
+				)
+				(hide yes)
+			)
+		)
+		(property "Cost (qty10)" "$0.090"
 			(at 180.34 83.82 0)
 			(effects
@@
 			)
 		)
-		(property "Cost" "$0.00"
+		(property "Cost" "$0.10"
 			(at 246.38 38.1 0)
 			(effects
@@
 			)
 		)
-		(property "RoHS Compliant" "NO"
+		(property "RoHS Compliant" "YES"
+			(at 246.38 38.1 0)
+			(effects
+				(font
+					(size 1.27 1.27)
+				)
+				(hide yes)
+			)
+		)
+		(property "Cost (qty10)" "$0.025"
 			(at 246.38 38.1 0)
 			(effects
@@
 			)
 		)
-		(property "Cost" "$0.00"
+		(property "Cost" "$0.10"
 			(at 226.06 142.24 0)
 			(effects
@@
 			)
 		)
-		(property "RoHS Compliant" "NO"
+		(property "RoHS Compliant" "YES"
+			(at 226.06 142.24 0)
+			(effects
+				(font
+					(size 1.27 1.27)
+				)
+				(hide yes)
+			)
+		)
+		(property "Cost (qty10)" "$0.025"
 			(at 226.06 142.24 0)
 			(effects
@@
 			)
 		)
-		(property "Cost" "$0.00"
+		(property "Cost" "$0.16"
 			(at 180.34 113.03 0)
 			(effects
@@
 			)
 		)
-		(property "RoHS Compliant" "NO"
+		(property "RoHS Compliant" "YES"
 			(at 180.34 113.03 0)
 			(effects
+				(font
+					(size 1.27 1.27)
+				)
+				(hide yes)
+			)
+		)
+		(property "Cost (qty10)" "$0.090"
+			(at 180.34 113.03 0)
+			(effects

Commit message: Almost done with generating bill of materials
Parts:
- R10, R8, R9: Cost $0.00 -> $0.10; Cost (qty10) (none) -> $0.030; RoHS Compliant NO -> YES
- R11: Cost $0.00 -> $2.05; Cost (qty10) (none) -> $1.732; RoHS Compliant NO -> YES
Changed lines of the file:
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@@
 			)
 		)
-		(property "Cost" "$0.00"
+		(property "Cost" "$0.10"
 			(at 220.98 59.69 0)
 			(effects
@@
 			)
 		)
-		(property "RoHS Compliant" "NO"
+		(property "RoHS Compliant" "YES"
+			(at 220.98 59.69 0)
+			(effects
+				(font
+					(size 1.27 1.27)
+				)
+				(hide yes)
+			)
+		)
+		(property "Cost (qty10)" "$0.030"
 			(at 220.98 59.69 0)
 			(effects
@@
 			)
 		)
-		(property "Cost" "$0.00"
+		(property "Cost" "$2.05"
 			(at 241.3 53.34 0)
 			(effects
@@
 			)
 		)
-		(property "RoHS Compliant" "NO"
+		(property "RoHS Compliant" "YES"
+			(at 241.3 53.34 0)
+			(effects
+				(font
+					(size 1.27 1.27)
+				)
+				(hide yes)
+			)
+		)
+		(property "Cost (qty10)" "$1.732"
 			(at 241.3 53.34 0)
 			(effects
@@
 			)
 		)
-		(property "Cost" "$0.00"
+		(property "Cost" "$0.10"
 			(at 220.98 107.95 0)
 			(effects
@@
 			)
 		)
-		(property "RoHS Compliant" "NO"
+		(property "RoHS Compliant" "YES"
+			(at 220.98 107.95 0)
+			(effects
+				(font
+					(size 1.27 1.27)
+				)
+				(hide yes)
+			)
+		)
+		(property "Cost (qty10)" "$0.030"
 			(at 220.98 107.95 0)
 			(effects
@@
 			)
 		)
-		(property "Cost" "$0.00"
+		(property "Cost" "$0.10"
 			(at 220.98 120.65 0)
 			(effects
@@
 			)
 		)
-		(property "RoHS Compliant" "NO"
+		(property "RoHS Compliant" "YES"
 			(at 220.98 120.65 0)
 			(effects
+				(font
+					(size 1.27 1.27)
+				)
+				(hide yes)
+			)
+		)
+		(property "Cost (qty10)" "$0.030"
+			(at 220.98 120.65 0)
+			(effects

Commit message: Starting major changes in response to the SOIC-8 version of OP37 being out of stock
Parts:
- U4: Cost $0.00 -> $3.47; Cost (qty10) (none) -> $2.30; Purchase Link https://www.digikey.com/en/products/detail/analog-devices-i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 -> https://www.mouser.com/ProductDetail/Analog-Devices/AD8615A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; RoHS Compliant NO -> YES
Changed lines of the file:
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@@
 			)
 		)
-		(property "Purchase Link" "https://www.digikey.com/en/products/detail/analog-devices-inc/AD8615AUJZ-REEL7/951437"
+		(property "Purchase Link" "https://www.mouser.com/ProductDetail/Analog-Devices/AD8615AUJZ-REEL?qs=%2FtpEQrCGXCx4ykDkhiJmqw%3D%3D"
 			(at 43.18 81.28 0)
 			(effects
@@
 			)
 		)
-		(property "Cost" "$0.00"
+		(property "Cost" "$3.47"
 			(at 43.18 81.28 0)
 			(effects
@@
 			)
 		)
-		(property "RoHS Compliant" "NO"
+		(property "RoHS Compliant" "YES"
 			(at 43.18 81.28 0)
 			(effects
+				(font
+					(size 1.27 1.27)
+				)
+				(hide yes)
+			)
+		)
+		(property "Cost (qty10)" "$2.30"
+			(at 43.18 81.28 0)
+			(effects

Commit message: Patching up the bill of materials now
Parts:
- U4: Cost $3.47 -> $0.00; Cost (qty10) $2.30 -> $0.00; Purchase Link https://www.mouser.com/ProductDetail/Analog-Devices/AD8615A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 -> (none)
Changed lines of the file:
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@@
 			)
 		)
-		(property "Purchase Link" "https://www.mouser.com/ProductDetail/Analog-Devices/AD8615AUJZ-REEL?qs=%2FtpEQrCGXCx4ykDkhiJmqw%3D%3D"
+		(property "Purchase Link" ""
 			(at 43.18 81.28 0)
 			(effects
@@
 			)
 		)
-		(property "Cost" "$3.47"
+		(property "Cost" "$0.00"
 			(at 43.18 81.28 0)
 			(effects
@@
 			)
 		)
-		(property "Cost (qty10)" "$2.30"
+		(property "Cost (qty10)" "$0.00"
 			(at 43.18 81.28 0)
 			(effects
