File: Models/TriangleWaveGenerator/DualOpAmp.kicad_sch (KiCad schematic)
At the start: 3 parts, among them U1 LF412CP

Commit message: Filled in breadboard schematic, now need purchase links
Connections:
- net Input1 renamed Input1(-)
Changed lines of the file:
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@@
 		)
 	)
-	(hierarchical_label "Input1"
+	(hierarchical_label "Input1(-)"
 		(shape input)
 		(at 121.92 83.82 180)

Commit message: Did the BOM
Parts:
- C1, C2: footprint (none) -> TwoTerminal:THT_2.54mm; Cost (none) -> $0.82; Cost (qty10) (none) -> $0.479; Purchase Link (none) -> https://www.digikey.com/en/products/detail/murata-electroni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; RoHS Compliant (none) -> YES
- U1: footprint P8 -> IC:PDIP-8; Cost (none) -> $1.57; Cost (qty10) (none) -> $1.145; Purchase Link (none) -> https://www.digikey.com/en/products/detail/texas-instrument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; RoHS Compliant (none) -> YES
Changed lines of the file:
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@@
 			)
 		)
-		(property "Footprint" ""
+		(property "Footprint" "TwoTerminal:THT_2.54mm"
 			(at 186.3852 78.74 0)
 			(effects
@@
 		)
 		(property "Description" "Unpolarized capacitor"
+			(at 185.42 74.93 0)
+			(effects
+				(font
+					(size 1.27 1.27)
+				)
+				(hide yes)
+			)
+		)
+		(property "Purchase Link" "https://www.digikey.com/en/products/detail/murata-electronics/RDE5C1H104J2P1H03B/10706775"
+			(at 185.42 74.93 0)
+			(effects
+				(font
+					(size 1.27 1.27)
+				)
+				(hide yes)
+			)
+		)
+		(property "Cost" "$0.82"
+			(at 185.42 74.93 0)
+			(effects
+				(font
+					(size 1.27 1.27)
+				)
+				(hide yes)
+			)
+		)
+		(property "Cost (qty10)" "$0.479"
+			(at 185.42 74.93 0)
+			(effects
+				(font
+					(size 1.27 1.27)
+				)
+				(hide yes)
+			)
+		)
+		(property "RoHS Compliant" "YES"
 			(at 185.42 74.93 0)
 			(effects
@@
 			)
 		)
-		(property "Footprint" "P8"
+		(property "Footprint" "IC:PDIP-8"
 			(at 121.92 81.28 0)
 			(effects
@@
 		)
 		(property "Description" ""
+			(at 121.92 81.28 0)
+			(effects
+				(font
+					(size 1.27 1.27)
+				)
+				(hide yes)
+			)
+		)
+		(property "Purchase Link" "https://www.digikey.com/en/products/detail/texas-instruments/LF412CP/378419"
+			(at 121.92 81.28 0)
+			(effects
+				(font
+					(size 1.27 1.27)
+				)
+				(hide yes)
+			)
+		)
+		(property "Cost" "$1.57"
+			(at 121.92 81.28 0)
+			(effects
+				(font
+					(size 1.27 1.27)
+				)
+				(hide yes)
+			)
+		)
+		(property "Cost (qty10)" "$1.145"
+			(at 121.92 81.28 0)
+			(effects
+				(font
+					(size 1.27 1.27)
+				)
+				(hide yes)
+			)
+		)
+		(property "RoHS Compliant" "YES"
 			(at 121.92 81.28 0)
 			(effects
@@
 			)
 		)
-		(property "Footprint" ""
+		(property "Footprint" "TwoTerminal:THT_2.54mm"
 			(at 115.2652 99.06 0)
 			(effects
@@
 			(at 114.3 95.25 0)
 			(effects
+				(font
+					(size 1.27 1.27)
+				)
+				(hide yes)
+			)
+		)
+		(property "Purchase Link" "https://www.digikey.com/en/products/detail/murata-electronics/RDE5C1H104J2P1H03B/10706775"
+			(at 114.3 95.25 0)
+			(effects
+				(font
+					(size 1.27 1.27)
+				)
+				(hide yes)
+			)
+		)
+		(property "Cost" "$0.82"
+			(at 114.3 95.25 0)
+			(effects
+				(font
+					(size 1.27 1.27)
+				)
+				(hide yes)
+			)
+		)
+		(property "Cost (qty10)" "$0.479"
+			(at 114.3 95.25 0)
+			(effects
+				(font
+					(size 1.27 1.27)
+				)
+				(hide yes)
+			)
+		)
+		(property "RoHS Compliant" "YES"
+			(at 114.3 95.25 0)
+			(effects
